Commit message: patched namespace and multi-robot issue

File: husky_description/urdf/decorations.urdf.xacro (robot description, xacro)
@@ -29,9 +29,9 @@
   <material name="white"><color rgba="1.0 1.0 1.0 1.0" /></material>
   <material name="red"><color rgba="1.0 0.0 0.0 1.0" /></material>
-  <xacro:macro name="husky_decorate">
+  <xacro:macro name="husky_decorate" params="namespace">
     <xacro:property name="husky_front_bumper_extend" value="$(optenv HUSKY_FRONT_BUMPER_EXTEND 0)" />
     <xacro:property name="husky_rear_bumper_extend" value="$(optenv HUSKY_REAR_BUMPER_EXTEND 0)" />
     <!-- Spawn Husky chassis -->
-    <link name="top_chassis_link">
+    <link name="${namespace}top_chassis_link">
       <visual>
         <origin xyz="0 0 0" rpy="0 0 0" />
@@ -42,11 +42,11 @@
     </link>
     <!-- Attach chassis to the robot -->
-    <joint name="top_chassis_joint" type="fixed">
-      <parent link="base_link" />
-      <child link="top_chassis_link" />
+    <joint name="${namespace}top_chassis_joint" type="fixed">
+      <parent link="${namespace}base_link" />
+      <child link="${namespace}top_chassis_link" />
     </joint>
     <xacro:if value="$(optenv HUSKY_USER_RAIL_ENABLED true)">
       <!-- Spawn user rails -->
-      <link name="user_rail_link">
+      <link name="${namespace}user_rail_link">
         <visual>
           <geometry>
@@ -56,12 +56,12 @@
       </link>
       <!-- Attach user rails to base link -->
-      <joint name="user_rail" type="fixed">
+      <joint name="${namespace}user_rail" type="fixed">
         <origin xyz="0.272 0 0.245" rpy="0 0 0" />
-        <parent link="base_link" />
-        <child link="user_rail_link" />
+        <parent link="${namespace}base_link" />
+        <child link="${namespace}user_rail_link" />
       </joint>
     </xacro:if>
     <!-- Spawn front bumper link -->
-    <link name="front_bumper_link">
+    <link name="${namespace}front_bumper_link">
       <visual>
         <geometry>
@@ -71,11 +71,11 @@
     </link>
     <!-- Attach front bumper -->
-    <joint name="front_bumper" type="fixed">
+    <joint name="${namespace}front_bumper" type="fixed">
       <origin xyz="${0.48 + husky_front_bumper_extend} 0 0.091" rpy="0 0 0" />
-      <parent link="base_link" />
-      <child link="front_bumper_link" />
+      <parent link="${namespace}base_link" />
+      <child link="${namespace}front_bumper_link" />
     </joint>
     <xacro:if value="${husky_front_bumper_extend}">
-      <link name="front_bumper_extension_link">
+      <link name="${namespace}front_bumper_extension_link">
           <visual>
               <geometry>
@@ -84,12 +84,12 @@
           </visual>
       </link>
-      <joint name="front_bumper_extension" type="fixed">
+      <joint name="${namespace}front_bumper_extension" type="fixed">
         <origin xyz="${0.48 + husky_front_bumper_extend} 0 0.091" rpy="0 0 0" />
-        <parent link="base_link" />
-        <child link="front_bumper_extension_link" />
+        <parent link="${namespace}base_link" />
+        <child link="${namespace}front_bumper_extension_link" />
       </joint>
     </xacro:if>
     <!-- Spawn rear bumper link -->
-    <link name="rear_bumper_link">
+    <link name="${namespace}rear_bumper_link">
       <visual>
         <geometry>
@@ -99,11 +99,11 @@
     </link>
     <!-- Attach rear bumper -->
-    <joint name="rear_bumper" type="fixed">
+    <joint name="${namespace}rear_bumper" type="fixed">
       <origin xyz="${-0.48 - husky_rear_bumper_extend} 0 0.091" rpy="0 0 ${M_PI}" />
-      <parent link="base_link" />
-      <child link="rear_bumper_link" />
+      <parent link="${namespace}base_link" />
+      <child link="${namespace}rear_bumper_link" />
     </joint>
     <xacro:if value="${husky_rear_bumper_extend}">
-      <link name="rear_bumper_extension_link">
+      <link name="${namespace}rear_bumper_extension_link">
           <visual>
               <geometry>
@@ -112,8 +112,8 @@
           </visual>
       </link>
-      <joint name="rear_bumper_extension" type="fixed">
+      <joint name="${namespace}rear_bumper_extension" type="fixed">
         <origin xyz="${-0.48 - husky_rear_bumper_extend} 0 0.091" rpy="0 0 ${M_PI}" />
-        <parent link="base_link" />
-        <child link="rear_bumper_extension_link" />
+        <parent link="${namespace}base_link" />
+        <child link="${namespace}rear_bumper_extension_link" />
       </joint>
     </xacro:if>
@@ -121,5 +121,5 @@
       <!-- Spawn the top plate -->
       <xacro:if value="$(optenv HUSKY_LARGE_TOP_PLATE false)">
-        <link name="top_plate_link">
+        <link name="${namespace}top_plate_link">
           <visual>
             <origin xyz="0 0 0" rpy="0 0 0" />
@@ -136,24 +136,24 @@
         </link>
         <!-- Attach top plate -->
-        <joint name="top_plate_joint" type="fixed">
-          <parent link="base_link" />
+        <joint name="${namespace}top_plate_joint" type="fixed">
+          <parent link="${namespace}base_link" />
           <child link="top_plate_link"/>
           <origin xyz="0.0812 0 0.225" rpy="0 0 0"/>
         </joint>
         <!-- Top plate front link -->
-        <joint name="top_plate_front_joint" type="fixed">
-          <parent link="top_plate_link" />
-          <child link="top_plate_front_link"/>
+        <joint name="${namespace}top_plate_front_joint" type="fixed">
+          <parent link="${namespace}top_plate_link" />
+          <child link="${namespace}top_plate_front_link"/>
           <origin xyz="0.4125 0 0.00672" rpy="0 0 0"/>
         </joint>
         <!-- Top plate rear link-->
-        <joint name="top_plate_rear_joint" type="fixed">
-          <parent link="top_plate_link" />
-          <child link="top_plate_rear_link"/>
+        <joint name="${namespace}top_plate_rear_joint" type="fixed">
+          <parent link="${namespace}top_plate_link" />
+          <child link="${namespace}top_plate_rear_link"/>
           <origin xyz="-0.4125 0 0.00672" rpy="0 0 0"/>
         </joint>
       </xacro:if>
       <xacro:unless value="$(optenv HUSKY_LARGE_TOP_PLATE false)">
-        <link name="top_plate_link">
+        <link name="${namespace}top_plate_link">
           <visual>
             <origin xyz="0 0 0" rpy="0 0 0" />
@@ -170,24 +170,24 @@
         </link>
         <!-- Attach top plate -->
-        <joint name="top_plate_joint" type="fixed">
-          <parent link="base_link" />
-          <child link="top_plate_link"/>
+        <joint name="${namespace}top_plate_joint" type="fixed">
+          <parent link="${namespace}base_link" />
+          <child link="${namespace}top_plate_link"/>
           <origin xyz="0.0812 0 0.245" rpy="0 0 0"/>
         </joint>
         <!-- Top plate front link -->
-        <joint name="top_plate_front_joint" type="fixed">
-          <parent link="top_plate_link" />
-          <child link="top_plate_front_link"/>
+        <joint name="${namespace}top_plate_front_joint" type="fixed">
+          <parent link="${namespace}top_plate_link" />
+          <child link="${namespace}top_plate_front_link"/>
           <origin xyz="0.36367 0 0.00639" rpy="0 0 0"/>
         </joint>
         <!-- Top plate rear link-->
-        <joint name="top_plate_rear_joint" type="fixed">
-          <parent link="top_plate_link" />
-          <child link="top_plate_rear_link"/>
+        <joint name="${namespace}top_plate_rear_joint" type="fixed">
+          <parent link="${namespace}top_plate_link" />
+          <child link="${namespace}top_plate_rear_link"/>
           <origin xyz="-0.36633 0 0.00639" rpy="0 0 0"/>
         </joint>
       </xacro:unless>
-      <link name="top_plate_front_link"/>
-      <link name="top_plate_rear_link"/>
+      <link name="${namespace}top_plate_front_link"/>
+      <link name="${namespace}top_plate_rear_link"/>
     </xacro:if>
   </xacro:macro>

File: husky_description/urdf/husky.urdf.xacro (robot description, xacro)
@@ -31,5 +31,6 @@
   <xacro:property name="husky_front_bumper_extend" value="$(optenv HUSKY_FRONT_BUMPER_EXTEND 0)" />
   <xacro:property name="husky_rear_bumper_extend" value="$(optenv HUSKY_REAR_BUMPER_EXTEND 0)" />
-  <xacro:arg name="robot_namespace" default="/" />
+  <xacro:arg name="namespace" default="" />
+  <xacro:arg name="suffix_ns" default="$(arg namespace)"/>
   <xacro:arg name="urdf_extras" default="empty.urdf" />
   <!-- Included URDF/XACRO Files -->
@@ -52,5 +53,5 @@
   <xacro:property name="wheel_radius" value="0.1651" />
   <!-- Base link is the center of the robot's bottom plate -->
-  <link name="base_link">
+  <link name="$(arg suffix_ns)base_link">
     <visual>
       <origin xyz="0 0 0" rpy="0 0 0" />
@@ -73,12 +74,12 @@
   </link>
   <!-- Base footprint is on the ground under the robot -->
-  <link name="base_footprint"/>
-  <joint name="base_footprint_joint" type="fixed">
+  <link name="$(arg suffix_ns)base_footprint"/>
+  <joint name="$(arg suffix_ns)base_footprint_joint" type="fixed">
     <origin xyz="0 0 ${wheel_vertical_offset - wheel_radius}" rpy="0 0 0" />
-    <parent link="base_link" />
-    <child link="base_footprint" />
+    <parent link="$(arg suffix_ns)base_link" />
+    <child link="$(arg suffix_ns)base_footprint" />
   </joint>
   <!-- Inertial link stores the robot's inertial information -->
-  <link name="inertial_link">
+  <link name="$(arg suffix_ns)inertial_link">
     <inertial>
       <mass value="46.034" />
@@ -87,109 +88,27 @@
     </inertial>
   </link>
-  <joint name="inertial_joint" type="fixed">
+  <joint name="$(arg suffix_ns)inertial_joint" type="fixed">
     <origin xyz="0 0 0" rpy="0 0 0" />
-    <parent link="base_link" />
-    <child link="inertial_link" />
+    <parent link="$(arg suffix_ns)base_link" />
+    <child link="$(arg suffix_ns)inertial_link" />
   </joint>
-  <!-- IMU Link is the standard mounting position for the UM6 IMU.-->
-  <!-- Can be modified with environment variables in /etc/ros/setup.bash -->
-  <link name="imu_link"/>
-  <joint name="imu_joint" type="fixed">
-    <origin xyz="$(optenv HUSKY_IMU_XYZ 0.19 0 0.149)" rpy="$(optenv HUSKY_IMU_RPY 0 -1.5708 3.1416)" />
-    <parent link="base_link" />
-    <child link="imu_link" />
-  </joint>
-  <gazebo reference="imu_link">
-  </gazebo>
   <!-- Husky wheel macros -->
-  <xacro:husky_wheel wheel_prefix="front_left">
+  <xacro:husky_wheel wheel_prefix="front_left" namespace="$(arg suffix_ns)">
     <origin xyz="${wheelbase/2} ${track/2} ${wheel_vertical_offset}" rpy="0 0 0" />
   </xacro:husky_wheel>
-  <xacro:husky_wheel wheel_prefix="front_right">
+  <xacro:husky_wheel wheel_prefix="front_right" namespace="$(arg suffix_ns)">
     <origin xyz="${wheelbase/2} ${-track/2} ${wheel_vertical_offset}" rpy="0 0 0" />
   </xacro:husky_wheel>
-  <xacro:husky_wheel wheel_prefix="rear_left">
+  <xacro:husky_wheel wheel_prefix="rear_left" namespace="$(arg suffix_ns)">
     <origin xyz="${-wheelbase/2} ${track/2} ${wheel_vertical_offset}" rpy="0 0 0" />
   </xacro:husky_wheel>
-  <xacro:husky_wheel wheel_prefix="rear_right">
+  <xacro:husky_wheel wheel_prefix="rear_right" namespace="$(arg suffix_ns)">
     <origin xyz="${-wheelbase/2} ${-track/2} ${wheel_vertical_offset}" rpy="0 0 0" />
   </xacro:husky_wheel>
-  <xacro:husky_decorate />
-  <xacro:if value="$(arg laser_enabled)">
-    <sick_lms1xx_mount prefix="base"/>
-    <sick_lms1xx frame="base_laser" topic="scan" robot_namespace="$(arg robot_namespace)"/>
-    <joint name="laser_mount_joint" type="fixed">
-      <origin xyz="$(arg laser_xyz)" rpy="$(arg laser_rpy)" />
-      <parent link="top_plate_link" />
-      <child link="base_laser_mount" />
-    </joint>
-  </xacro:if>
-  <!--
-    top sensor arch; include this if we have realsense enabled
-    keep this as a property to make it easier to add multiple conditions, should we need
-    the top bar for any additional sensors in the future
-  -->
-  <xacro:property name="topbar_needed_realsense" value="$(arg realsense_enabled)" />
-  <xacro:if value="${topbar_needed_realsense}">
-    <xacro:sensor_arch prefix="" parent="top_plate_link">
-      <origin xyz="-0.35 0 0.51" rpy="0 0 -3.14"/>
-    </xacro:sensor_arch>
-  </xacro:if>
-  <!-- add the intel realsense to the topbar if needed -->
-  <xacro:if value="$(arg realsense_enabled)">
-    <link name="realsense_mountpoint"/>
-    <joint name="realsense_mountpoint_joint" type="fixed">
-      <origin xyz="0 0 0" rpy="0 0 -3.14159" />
-      <parent link="$(arg realsense_mount)"/>
-      <child link="realsense_mountpoint" />
-    </joint>
-    <xacro:intel_realsense_mount prefix="camera" topic="realsense" parent_link="realsense_mountpoint"/>
-  </xacro:if>
-  <gazebo>
-    <plugin name="gazebo_ros_control" filename="libgazebo_ros_control.so">
-      <robotNamespace>$(arg robot_namespace)</robotNamespace>
-      <legacyModeNS>true</legacyModeNS>
-    </plugin>
-  </gazebo>
-  <gazebo>
-    <plugin name="imu_controller" filename="libhector_gazebo_ros_imu.so">
-      <robotNamespace>$(arg robot_namespace)</robotNamespace>
-      <updateRate>50.0</updateRate>
-      <bodyName>base_link</bodyName>
-      <topicName>imu/data</topicName>
-      <accelDrift>0.005 0.005 0.005</accelDrift>
-      <accelGaussianNoise>0.005 0.005 0.005</accelGaussianNoise>
-      <rateDrift>0.005 0.005 0.005 </rateDrift>
-      <rateGaussianNoise>0.005 0.005 0.005 </rateGaussianNoise>
-      <headingDrift>0.005</headingDrift>
-      <headingGaussianNoise>0.005</headingGaussianNoise>
-    </plugin>
-  </gazebo>
-  <gazebo>
-    <plugin name="gps_controller" filename="libhector_gazebo_ros_gps.so">
-      <robotNamespace>$(arg robot_namespace)</robotNamespace>
-      <updateRate>40</updateRate>
-      <bodyName>base_link</bodyName>
-      <frameId>base_link</frameId>
-      <topicName>navsat/fix</topicName>
-      <velocityTopicName>navsat/vel</velocityTopicName>
-      <referenceLatitude>49.9</referenceLatitude>
-      <referenceLongitude>8.9</referenceLongitude>
-      <referenceHeading>0</referenceHeading>
-      <referenceAltitude>0</referenceAltitude>
-      <drift>0.0001 0.0001 0.0001</drift>
-    </plugin>
-  </gazebo>
-  <!-- Mount a Perfect Pose 3D sensor. -->
-  <gazebo>
-    <plugin filename="libgazebo_ros_p3d.so" name="groundtruth_sim">
-      <updateRate>50.0</updateRate>
-      <robotNamespace>/$(arg robot_namespace)</robotNamespace>
-      <bodyName>base_link</bodyName>
-      <topicName>/pose_gt</topicName>
-      <gaussianNoise>0.0</gaussianNoise>
-      <frameName>world</frameName>
-    </plugin>
-  </gazebo>
+  <!-- Includes bumpers and other cosmetics -->
+  <xacro:husky_decorate namespace="$(arg suffix_ns)" />
+  <!-- Include the sensor modules -->
+  <xacro:include filename="$(find husky_description)/urdf/accessories.urdf.xacro"/>
+  <xacro:include filename="$(find husky_description)/urdf/sensors.xacro"/>
   <!-- Optional custom includes. -->
   <xacro:include filename="$(arg urdf_extras)" />

File: husky_description/urdf/wheel.urdf.xacro (robot description, xacro)
@@ -22,6 +22,6 @@
 -->
 <robot xmlns:xacro="http://ros.org/wiki/xacro" name="husky_wheel">
-	<xacro:macro name="husky_wheel" params="wheel_prefix *joint_pose">
-		<link name="${wheel_prefix}_wheel_link">
+	<xacro:macro name="husky_wheel" params="namespace wheel_prefix *joint_pose">
+		<link name="${namespace}${wheel_prefix}_wheel_link">
 			<inertial>
 				<mass value="2.637" />
@@ -42,5 +42,5 @@
 			</collision>
 		</link>
-		<gazebo reference="${wheel_prefix}_wheel_link">
+		<gazebo reference="${namespace}${wheel_prefix}_wheel_link">
 			<mu1 value="1.0"/>
 			<mu2 value="1.0"/>
@@ -49,16 +49,16 @@
 			<fdir1 value="1 0 0"/>
 		</gazebo>
-		<joint name="${wheel_prefix}_wheel" type="continuous">
-			<parent link="base_link"/>
-			<child link="${wheel_prefix}_wheel_link"/>
+		<joint name="${namespace}${wheel_prefix}_wheel" type="continuous">
+			<parent link="${namespace}base_link"/>
+			<child link="${namespace}${wheel_prefix}_wheel_link"/>
 			<xacro:insert_block name="joint_pose"/>
 			<axis xyz="0 1 0" rpy="0 0 0" />
 		</joint>
-		<transmission name="${wheel_prefix}_wheel_trans" type="SimpleTransmission">
+		<transmission name="${namespace}${wheel_prefix}_wheel_trans" type="SimpleTransmission">
 			<type>transmission_interface/SimpleTransmission</type>
-			<actuator name="${wheel_prefix}_wheel_motor">
+			<actuator name="${namespace}${wheel_prefix}_wheel_motor">
 				<mechanicalReduction>1</mechanicalReduction>
 			</actuator>
-			<joint name="${wheel_prefix}_wheel">
+			<joint name="${namespace}${wheel_prefix}_wheel">
 				<hardwareInterface>hardware_interface/VelocityJointInterface</hardwareInterface>
 			</joint>
