Commit message: drive husky with rear wheels

File: husky_description/urdf/accessories/os1.urdf.xacro (robot description, xacro)
@@ -11,8 +11,13 @@
     <link name="${frame}">
       <inertial>
-         <mass value="0.33"/>
+        <mass value="1.1" />
+        <origin xyz="0 0 0" />
+        <inertia ixx="${0.0833333 * 1.1 * (0.102*0.102 + 0.152*0.152)}" ixy="0.0" ixz="0.0"
+          iyy="${0.0833333 * 1.1 * (0.105*0.105 + 0.152*0.152)}" iyz="0.0"
+          izz="${0.0833333 * 1.1 * (0.105*0.105 + 0.102*0.102)}" />
+         <!--mass value="0.33"/>
          <origin xyz="0 0 0.0365" rpy="0 0 0" />
          <inertia ixx="0.000241148" ixy="0" ixz="0"
-          iyy="0.000241148" iyz="0" izz="0.000264"/>
+          iyy="0.000241148" iyz="0" izz="0.000264"/-->
       </inertial>
       <collision name="base_collision">

File: husky_description/urdf/base.xacro (robot description, xacro)
@@ -82,14 +82,14 @@
     </joint>
     <!-- Husky wheel macros -->
-    <xacro:husky_wheel wheel_prefix="front_left" namespace="${namespace}">
+    <xacro:husky_wheel wheel_prefix="front_left" drive="false" namespace="${namespace}">
       <origin xyz="${wheelbase/2} ${track/2} ${wheel_vertical_offset}" rpy="0 0 0" />
     </xacro:husky_wheel>
-    <xacro:husky_wheel wheel_prefix="front_right" namespace="${namespace}">
+    <xacro:husky_wheel wheel_prefix="front_right" drive="false" namespace="${namespace}">
       <origin xyz="${wheelbase/2} ${-track/2} ${wheel_vertical_offset}" rpy="0 0 0" />
     </xacro:husky_wheel>
-    <xacro:husky_wheel wheel_prefix="rear_left" namespace="${namespace}">
+    <xacro:husky_wheel wheel_prefix="rear_left" drive="true" namespace="${namespace}">
       <origin xyz="${-wheelbase/2} ${track/2} ${wheel_vertical_offset}" rpy="0 0 0" />
     </xacro:husky_wheel>
-    <xacro:husky_wheel wheel_prefix="rear_right" namespace="${namespace}">
+    <xacro:husky_wheel wheel_prefix="rear_right" drive="true" namespace="${namespace}">
       <origin xyz="${-wheelbase/2} ${-track/2} ${wheel_vertical_offset}" rpy="0 0 0" />
     </xacro:husky_wheel>

File: husky_description/urdf/wheel.urdf.xacro (robot description, xacro)
@@ -22,5 +22,5 @@
 -->
 <robot xmlns:xacro="http://ros.org/wiki/xacro" name="husky_wheel">
-	<xacro:macro name="husky_wheel" params="namespace wheel_prefix *joint_pose">
+	<xacro:macro name="husky_wheel" params="namespace wheel_prefix drive *joint_pose">
 		<link name="${namespace}${wheel_prefix}_wheel_link">
 			<inertial>
@@ -42,10 +42,19 @@
 			</collision>
 		</link>
-		<gazebo reference="${namespace}${wheel_prefix}_wheel_link">
-			<mu1 value="1.0"/>
-			<mu2 value=".5"/>
-			<kp value="10000000.0" />
-			<kd value="1.0" />
-			<fdir1 value="1 0 0"/>
+        <gazebo reference="${namespace}${wheel_prefix}_wheel_link">
+            <xacro:if value="${drive}">
+		    	<mu1 value="1.0"/>
+		    	<mu2 value=".5"/>
+		    	<kp value="10000000.0" />
+		    	<kd value="1.0" />
+		    	<fdir1 value="1 0 0"/>
+            </xacro:if>
+            <xacro:unless value="${drive}">
+		    	<mu1 value=".0"/>
+		    	<mu2 value=".0"/>
+		    	<kp value="10000000.0" />
+		    	<kd value="1.0" />
+		    	<fdir1 value="1 0 0"/>
+            </xacro:unless>
 		</gazebo>
 		<joint name="${namespace}${wheel_prefix}_wheel" type="continuous">
@@ -55,13 +64,15 @@
 			<axis xyz="0 1 0" rpy="0 0 0" />
 		</joint>
-		<transmission name="${namespace}${wheel_prefix}_wheel_trans" type="SimpleTransmission">
-			<type>transmission_interface/SimpleTransmission</type>
-			<actuator name="${namespace}${wheel_prefix}_wheel_motor">
-				<mechanicalReduction>1</mechanicalReduction>
-			</actuator>
-			<joint name="${namespace}${wheel_prefix}_wheel">
-				<hardwareInterface>hardware_interface/VelocityJointInterface</hardwareInterface>
-			</joint>
-		</transmission>
+        <xacro:if value="${drive}">
+            <transmission name="${namespace}${wheel_prefix}_wheel_trans" type="SimpleTransmission">
+                <type>transmission_interface/SimpleTransmission</type>
+                <actuator name="${namespace}${wheel_prefix}_wheel_motor">
+                    <mechanicalReduction>1</mechanicalReduction>
+                </actuator>
+                <joint name="${namespace}${wheel_prefix}_wheel">
+                    <hardwareInterface>hardware_interface/VelocityJointInterface</hardwareInterface>
+                </joint>
+            </transmission>
+        </xacro:if>
 	</xacro:macro>
 </robot>
